Commit message: Update trinamic_urdf.urdf.xacro

File: urdf/trinamic_urdf.urdf.xacro (robot description, xacro)
@@ -1,13 +1,4 @@
 <?xml version="1.0"?>
 <robot name="trinamic" xmlns:xacro="http://ros.org/wiki/xacro">
-   <material name="blue">
-	  <color rgba="0 0 0.8 1"/>
-   </material>
-   <material name="green">
-      <color rgba="0.0 0.8 0.0 1.0"/>
-   </material>
-   <material name="white">
-	<color rgba="1 1 1 1"/>
-   </material>
   <link name="world">
    </link>
@@ -15,57 +6,22 @@
      <origin rpy="0 0 0" xyz="0 0 0"/>
      <parent link="world"/>
-     <child link="motor"/>
+     <child link="shaft"/>
    </joint>
-   <link name="motor">
-   <visual>
-      <geometry>
-          <cylinder length="0.035" radius="0.009"/>
-      </geometry>
-      <material name="white"/>
-      <origin rpy="0 1.5708 0" xyz="0 0 0.01"/>
-    </visual>
+   <link name="shaft">
    </link>
    <joint name="fixed_joint" type="fixed">
      <origin rpy="0 0 0" xyz="0.0175 0 0.01"/>
-     <parent link="motor"/>
-     <child link="motor_gear_box"/>
+     <parent link="shaft"/>
+     <child link="shaft2"/>
    </joint>
-  <link name="motor_gear_box">
-   <visual>
-      <geometry>
-         <box size="0.045 0.035 0.02"/>
-      </geometry>
-      <material name="white"/>
-      <origin rpy="0 0 0" xyz="0.0225 0 0"/>
-    </visual>
+  <link name="shaft2">
    </link>
    <joint name="servo1" type="continuous">
      <axis xyz="0 0 1"/>
      <origin rpy="0 0 0" xyz="0.02 0 0.01"/>
-     <parent link="motor_gear_box"/>
-     <child link="shaft"/>
+     <parent link="shaft2"/>
+     <child link="ghost"/>
    </joint>
-   <link name="shaft">
-   <visual>
-      <geometry>
-         <cylinder length="0.02" radius="0.002"/>
-      </geometry>
-      <material name="green"/>
-      <origin rpy="0 0 0" xyz="0 0 0.01"/>
-    </visual>
-   </link>
-   <joint name="shaft_joint" type="fixed">
-     <origin rpy="0 0 0" xyz="0.0 0 0.02"/>
-     <parent link="shaft"/>
-     <child link="shaft_bar"/>
-   </joint>
-   <link name="shaft_bar">
-   <visual>
-      <geometry>
-         <box size="0.05 0.02 0.001"/>
-      </geometry>
-      <material name="blue"/>
-      <origin rpy="0 0 0" xyz="0.015 0 0"/>
-    </visual>
+   <link name="ghost">
    </link>
  </robot>
